File: 回路図/オプトエレクトロニクス回路案_v2.kicad_sch (KiCad schematic)
At the start: 159 parts, among them J301 OUTPUT, J401 INPUT, Q301 2SC945-K, Q401 2SC2240-GR, SW101 SW_SPDT_MSM, SW301 SW_SPDT_MSM, SW302 SW_SPST, SW303 SW_SPST, U101 78L05, U103 NJU7032D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

Commit message: 回路Aの修正
Connections:
- net at R107.1, U105.1: now also U105.2 (-); no longer U105.3 (+)
- net at C106.1, RV101.2: now also U105.3 (+); no longer U105.2 (-)
Changed lines of the file:
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@@
 		(lib_id "Amplifier_Operational:NJM4580")
 		(at 154.94 48.26 0)
+		(mirror x)
 		(unit 1)
 		(exclude_from_sim no)
@@
 		(dnp no)
 		(property "Reference" "U105"
-			(at 155.956 51.308 0)
+			(at 156.21 51.562 0)
 			(effects
 				(font
@@
 		)
 		(property "Value" "NJU7032D"
-			(at 152.4 53.848 0)
+			(at 156.21 53.848 0)
 			(effects
 				(font
